Commit message: add h12 magpie urdf

File: unitree_robots/h1_2/h1_2_magpie.urdf (robot description, URDF)
Before this commit: robot h1_2, 34 links, 33 joints
Links:
- link left_ankle_pitch_link: geometry visual mesh filename=meshes/left_ankle_pitch_link.STL
- link left_ankle_roll_link: geometry collision mesh filename=meshes/left_ankle_roll_link.STL; visual mesh filename=meshes/left_ankle_roll_link.STL
- link left_elbow_link: geometry collision mesh filename=meshes/left_elbow_link.STL; visual mesh filename=meshes/left_elbow_link.STL
- link left_hip_pitch_link: geometry collision mesh filename=meshes/left_hip_pitch_link.STL; visual mesh filename=meshes/left_hip_pitch_link.STL
- link left_hip_roll_link: geometry collision mesh filename=meshes/left_hip_roll_link.STL; visual mesh filename=meshes/left_hip_roll_link.STL
- link left_hip_yaw_link: geometry visual mesh filename=meshes/left_hip_yaw_link.STL
- link left_knee_link: geometry collision cylinder length=0.2 radius=0.04; visual mesh filename=meshes/left_knee_link.STL
- link left_shoulder_pitch_link: geometry collision mesh filename=meshes/left_shoulder_pitch_link.STL; visual mesh filename=meshes/left_shoulder_pitch_link.STL
- link left_shoulder_roll_link: geometry collision mesh filename=meshes/left_shoulder_roll_link.STL; visual mesh filename=meshes/left_shoulder_roll_link.STL
- link left_shoulder_yaw_link: geometry collision mesh filename=meshes/left_shoulder_yaw_link.STL; visual mesh filename=meshes/left_shoulder_yaw_link.STL
- link left_wrist_pitch_link: geometry collision mesh filename=meshes/left_wrist_pitch_link.STL; visual mesh filename=meshes/left_wrist_pitch_link.STL
- link left_wrist_roll_link: geometry collision mesh filename=meshes/left_wrist_roll_link.STL; visual mesh filename=meshes/left_wrist_roll_link.STL
- link left_wrist_yaw_link: geometry collision cylinder length=0.02500000 radius=0.03200000; visual mesh filename=meshes/magpie/magpie_h12.stl scale=0.001 0.001 0.001
- link logo_link: geometry visual mesh filename=meshes/logo_link.STL
- link pelvis: geometry collision mesh filename=meshes/pelvis.STL; visual mesh filename=meshes/pelvis.STL
- link right_ankle_pitch_link: geometry visual mesh filename=meshes/right_ankle_pitch_link.STL
- link right_ankle_roll_link: geometry collision mesh filename=meshes/right_ankle_roll_link.STL; visual mesh filename=meshes/right_ankle_roll_link.STL
- link right_elbow_link: geometry collision mesh filename=meshes/right_elbow_link.STL; visual mesh filename=meshes/right_elbow_link.STL
- link right_hip_pitch_link: geometry collision mesh filename=meshes/right_hip_pitch_link.STL; visual mesh filename=meshes/right_hip_pitch_link.STL
- link right_hip_roll_link: geometry collision mesh filename=meshes/right_hip_roll_link.STL; visual mesh filename=meshes/right_hip_roll_link.STL
- link right_hip_yaw_link: geometry visual mesh filename=meshes/right_hip_yaw_link.STL
- link right_knee_link: geometry collision cylinder length=0.2 radius=0.04; visual mesh filename=meshes/right_knee_link.STL
- link right_shoulder_pitch_link: geometry collision mesh filename=meshes/right_shoulder_pitch_link.STL; visual mesh filename=meshes/right_shoulder_pitch_link.STL
- link right_shoulder_roll_link: geometry collision mesh filename=meshes/right_shoulder_roll_link.STL; visual mesh filename=meshes/right_shoulder_roll_link.STL
- link right_shoulder_yaw_link: geometry collision mesh filename=meshes/right_shoulder_yaw_link.STL; visual mesh filename=meshes/right_shoulder_yaw_link.STL
- link right_wrist_pitch_link: geometry collision mesh filename=meshes/right_wrist_pitch_link.STL; visual mesh filename=meshes/right_wrist_pitch_link.STL
- link right_wrist_roll_link: geometry collision mesh filename=meshes/right_wrist_roll_link.STL; visual mesh filename=meshes/right_wrist_roll_link.STL
- link right_wrist_yaw_link: geometry collision cylinder length=0.02500000 radius=0.03200000; visual mesh filename=meshes/magpie/magpie_h12.stl scale=0.001 0.001 0.001
- link torso_link: geometry collision mesh filename=meshes/torso_link.STL; visual mesh filename=meshes/torso_link.STL
