Commit message: Update model description file

File: unitree_robots/h1_2/h1_2.urdf (robot description, URDF)
Before this commit: robot h1_5, 56 links, 55 joints
Links:
- removed link left_elbow_pitch_link
- removed link left_elbow_roll_link
- removed link right_elbow_pitch_link
- removed link right_elbow_roll_link
- added link camera_link
- added link left_elbow_link, mass 0.691; collision mesh filename=meshes/left_elbow_link.STL; visual mesh filename=meshes/left_elbow_link.STL
- added link left_wrist_roll_link, mass 0.683; collision mesh filename=meshes/left_wrist_roll_link.STL; visual mesh filename=meshes/left_wrist_roll_link.STL
- added link lidar_link
- added link right_elbow_link, mass 0.691; collision mesh filename=meshes/right_elbow_link.STL; visual mesh filename=meshes/right_elbow_link.STL
- added link right_wrist_roll_link, mass 0.683; collision mesh filename=meshes/right_wrist_roll_link.STL; visual mesh filename=meshes/right_wrist_roll_link.STL
Joints:
- removed joint left_elbow_pitch_joint
- removed joint left_elbow_roll_joint
- removed joint right_elbow_pitch_joint
- removed joint right_elbow_roll_joint
- added joint camera_joint: type fixed, parent torso_link, child camera_link, origin xyz=0.11109 0.01750 0.68789 rpy=0 0.8859291283123216 0
- added joint left_elbow_joint: type revolute, parent left_shoulder_yaw_link, child left_elbow_link, origin xyz=0.006 0.0329 -0.182 rpy=0 0 0, axis 0 1 0, limit lower=-0.95 upper=3.18 effort=18 velocity=20
- added joint left_wrist_roll_joint: type revolute, parent left_elbow_link, child left_wrist_roll_link, origin xyz=0.121 -0.0329 -0.011 rpy=0 0 0, axis 1 0 0, limit lower=-3.01 upper=2.75 effort=19 velocity=31.4
- added joint lidar_joint: type fixed, parent torso_link, child lidar_link, origin xyz=0.04874 0 0.67980 rpy=0 0.24015730507441985 0
- added joint right_elbow_joint: type revolute, parent right_shoulder_yaw_link, child right_elbow_link, origin xyz=0.006 -0.0329 -0.182 rpy=0 0 0, axis 0 1 0, limit lower=-0.95 upper=3.18 effort=18 velocity=20
- added joint right_wrist_roll_joint: type revolute, parent right_elbow_link, child right_wrist_roll_link, origin xyz=0.121 0.0329 -0.011 rpy=0 0 0, axis 1 0 0, limit lower=-2.75 upper=3.01 effort=19 velocity=31.4
- joint imu_joint: origin xyz=-0.04233868314 0.00166 0.152067 rpy=0 0 0 -> xyz=-0.04452 -0.01891 0.27756 rpy=0 0 0
- joint left_knee_joint: limit lower=-0.26 upper=2.05 effort=300 velocity=14 -> lower=-0.12 upper=2.19 effort=300 velocity=14
- joint left_wrist_pitch_joint: limit lower=-0.47 upper=0.47 effort=19 velocity=31.4 -> lower=-0.4625 upper=0.4625 effort=19 velocity=31.4; origin xyz=0.085 0 0 rpy=0 0 0 -> xyz=0.087 0 0 rpy=0 0 0; parent left_elbow_roll_link -> left_wrist_roll_link
- joint right_knee_joint: limit lower=-0.26 upper=2.05 effort=300 velocity=14 -> lower=-0.12 upper=2.19 effort=300 velocity=14
- joint right_wrist_pitch_joint: limit lower=-0.47 upper=0.47 effort=19 velocity=31.4 -> lower=-0.4625 upper=0.4625 effort=19 velocity=31.4; origin xyz=0.085 0 0 rpy=0 0 0 -> xyz=0.087 0 0 rpy=0 0 0; parent right_elbow_roll_link -> right_wrist_roll_link

Commit message: Sync changes from h12_ros2_model

File: unitree_robots/h1_2/h1_2.urdf (robot description, URDF)
Before this commit: robot h1_2, 58 links, 57 joints
Links:
- removed link camera_link
- added link head_camera_link
- added link left_hand_camera_link
- added link right_hand_camera_link
Joints:
- removed joint camera_joint
- added joint head_camera_joint: type fixed, parent torso_link, child head_camera_link, origin xyz=0.11109 0.01750 0.68789 rpy=-2.45672546 0 -1.5708
- added joint left_hand_camera_joint: type fixed, parent left_wrist_yaw_link, child left_hand_camera_link, origin xyz=0 0.04 0 rpy=0 1.5708 0
- added joint right_hand_camera_joint: type fixed, parent right_wrist_yaw_link, child right_hand_camera_link, origin xyz=0 -0.04 0 rpy=-3.1415 -1.5708 0
- joint lidar_joint: origin xyz=0.04874 0 0.67980 rpy=0 0.24015730507441985 0 -> xyz=0.04874 0 0.679808 rpy=0 -2.90143535 0

Commit message: going to test single rollout

File: unitree_robots/h1_2/h1_2.urdf (robot description, URDF)
Before this commit: robot h1_2, 60 links, 59 joints
Joints:
- joint right_shoulder_roll_joint: limit lower=-3.4 upper=0.38 effort=40 velocity=9 -> lower=-3.4 upper=0.19 effort=40 velocity=9

File: unitree_robots/h1_2/h1_2_handless.urdf (robot description, URDF)
Before this commit: robot h1_2, 32 links, 31 joints
Joints:
- joint right_shoulder_roll_joint: limit lower=-3.4 upper=0.38 effort=40 velocity=9 -> lower=-3.4 upper=0.19 effort=40 velocity=9
